File: pandora/pandora.kicad_pcb (KiCad board)
At the start: 2 copper layers, 0 parts

Commit message: Start layout
Parts:
- added AE1: SWRU120D, pandora:Texas_SWRU120D_InvF_2.4GHz, F.Cu at (129.2, 68.3)
- added C1: 0.1uF, Capacitor_SMD:C_0603_1608Metric_Pad1.05x0.95mm_HandSolder, F.Cu at (212.1, 33.0)
- added C10: 22uF, Capacitor_SMD:C_0805_2012Metric_Pad1.15x1.40mm_HandSolder, F.Cu at (178.0, 36.1)
- added C11: 1uF, Capacitor_SMD:C_0603_1608Metric_Pad1.05x0.95mm_HandSolder, F.Cu at (225.4, -72.4)
- added C12: 1uF, Capacitor_SMD:C_0603_1608Metric_Pad1.05x0.95mm_HandSolder, F.Cu at (237.5, -74.3)
- added C13: 10uF, Capacitor_SMD:C_0805_2012Metric_Pad1.15x1.40mm_HandSolder, F.Cu at (188.4, 26.7)
- added C14: 1uF, Capacitor_SMD:C_0603_1608Metric_Pad1.05x0.95mm_HandSolder, F.Cu at (225.4, -66.0)
- added C15: 1uF, Capacitor_SMD:C_0603_1608Metric_Pad1.05x0.95mm_HandSolder, F.Cu at (237.5, -67.9)
- added C16: 0.1uF, Capacitor_SMD:C_0603_1608Metric_Pad1.05x0.95mm_HandSolder, F.Cu at (293.4, -48.3)
- added C17: 1uF, Capacitor_SMD:C_0603_1608Metric_Pad1.05x0.95mm_HandSolder, F.Cu at (285.1, -52.7)
- added C18: 10nF, Capacitor_SMD:C_0603_1608Metric_Pad1.05x0.95mm_HandSolder, F.Cu at (123.2, 92.7)
- added C19: 0.1uF, Capacitor_SMD:C_0603_1608Metric_Pad1.05x0.95mm_HandSolder, F.Cu at (114.3, 92.7)
- added C2: 1uF, Capacitor_SMD:C_0603_1608Metric_Pad1.05x0.95mm_HandSolder, F.Cu at (214.6, 33.0)
- added C20: 0.1uF, Capacitor_SMD:C_0603_1608Metric_Pad1.05x0.95mm_HandSolder, F.Cu at (119.4, 96.5)
- added C21: 0.1uF, Capacitor_SMD:C_0603_1608Metric_Pad1.05x0.95mm_HandSolder, F.Cu at (237.5, 49.5)
- added C22: 12pF, pandora:0402_HandSoldering, F.Cu at (138.6, 73.4)
- added C23: 1.8pF, pandora:0402_HandSoldering, F.Cu at (147.2, 64.9)
- added C24: 1pF, pandora:0402_HandSoldering, F.Cu at (135.5, 75.4)
- added C25: 12pF, pandora:0402_HandSoldering, F.Cu at (144.0, 66.8)
- added C26: 1pF, pandora:0402_HandSoldering, F.Cu at (135.5, 73.4)
- added C27: 1pF, pandora:0402_HandSoldering, F.Cu at (144.0, 64.9)
- added C28: 0.1uF, Capacitor_SMD:C_0603_1608Metric_Pad1.05x0.95mm_HandSolder, F.Cu at (174.7, 90.4)
- added C29: 0.1uF, Capacitor_SMD:C_0603_1608Metric_Pad1.05x0.95mm_HandSolder, F.Cu at (186.3, 72.3)
- added C3: 10uF, Capacitor_SMD:C_0805_2012Metric_Pad1.15x1.40mm_HandSolder, F.Cu at (217.2, 33.0)
- added C30: 0.1uF, Capacitor_SMD:C_0603_1608Metric_Pad1.05x0.95mm_HandSolder, F.Cu at (180.1, 78.2)
- added C31: 0.1uF, Capacitor_SMD:C_0603_1608Metric_Pad1.05x0.95mm_HandSolder, F.Cu at (182.0, 74.9)
- added C32: 22uF, Capacitor_SMD:C_0805_2012Metric_Pad1.15x1.40mm_HandSolder, F.Cu at (182.5, 67.1)
- added C33: 0.1uF, Capacitor_SMD:C_0603_1608Metric_Pad1.05x0.95mm_HandSolder, F.Cu at (182.0, 72.3)
- added C34: 22uF, Capacitor_SMD:C_0805_2012Metric_Pad1.15x1.40mm_HandSolder, F.Cu at (171.2, 79.1)
- added C35: 0.1uF, Capacitor_SMD:C_0603_1608Metric_Pad1.05x0.95mm_HandSolder, F.Cu at (177.6, 75.6)
- added C36: 0.1uF, Capacitor_SMD:C_0603_1608Metric_Pad1.05x0.95mm_HandSolder, F.Cu at (177.6, 73.1)
- added C37: 1uF, Capacitor_SMD:C_0603_1608Metric_Pad1.05x0.95mm_HandSolder, F.Cu at (187.0, 66.4)
- added C38: 15pF, Capacitor_SMD:C_0603_1608Metric_Pad1.05x0.95mm_HandSolder, F.Cu at (184.5, 69.8)
- added C39: 15pF, Capacitor_SMD:C_0603_1608Metric_Pad1.05x0.95mm_HandSolder, F.Cu at (175.7, 78.9)
- added C4: 47uF, Capacitor_SMD:C_1210_3225Metric_Pad1.42x2.65mm_HandSolder, F.Cu at (174.6, -12.7)
- added C40: 12pF, pandora:0402_Branch_HandSoldering, F.Cu at (190.2, 64.8)
- added C41: 12pF, pandora:0402_Branch_HandSoldering, F.Cu at (189.5, 72.3)
- added C42: 0.1uF, Capacitor_SMD:C_0603_1608Metric_Pad1.05x0.95mm_HandSolder, F.Cu at (188.8, 69.0)
- added C43: 0.1uF, Capacitor_SMD:C_0603_1608Metric_Pad1.05x0.95mm_HandSolder, F.Cu at (186.3, 74.9)
- added C44: 4.7uF, Capacitor_SMD:C_0805_2012Metric_Pad1.15x1.40mm_HandSolder, F.Cu at (208.8, 71.0)
- added C45: 4.7uF, Capacitor_SMD:C_0805_2012Metric_Pad1.15x1.40mm_HandSolder, F.Cu at (216.7, 62.5)
- added C46: 4.7uF, Capacitor_SMD:C_0805_2012Metric_Pad1.15x1.40mm_HandSolder, F.Cu at (252.1, 54.0)
- added C47: 0.1uF, Capacitor_SMD:C_0603_1608Metric_Pad1.05x0.95mm_HandSolder, F.Cu at (246.4, 60.3)
- added C48: 1uF, Capacitor_SMD:C_0603_1608Metric_Pad1.05x0.95mm_HandSolder, F.Cu at (246.4, 62.2)
- added C49: 10uF, Capacitor_SMD:C_0805_2012Metric_Pad1.15x1.40mm_HandSolder, F.Cu at (246.4, 64.1)
- added C5: 1uF, Capacitor_SMD:C_0603_1608Metric_Pad1.05x0.95mm_HandSolder, F.Cu at (171.4, -12.7)
- added C6: 0.1uF, Capacitor_SMD:C_0603_1608Metric_Pad1.05x0.95mm_HandSolder, F.Cu at (168.9, -12.7)
- added C7: 47uF, Capacitor_Tantalum_SMD:CP_EIA-7343-31_Kemet-D, F.Cu at (186.8, 12.6)
- added C8: 10uF, Capacitor_Tantalum_SMD:CP_EIA-7132-28_AVX-C_Pad2.72x3.50mm_HandSolder, F.Cu at (328.9, -33.0)
- added C9: 10uF, Capacitor_Tantalum_SMD:CP_EIA-7132-28_AVX-C_Pad2.72x3.50mm_HandSolder, F.Cu at (323.9, -40.6)
- added D1: S3JBHR5G, Diode_SMD:D_SMB_Handsoldering, F.Cu at (182.2, -11.4)
- added D10: RED, LED_SMD:LED_0805_2012Metric_Pad1.15x1.40mm_HandSolder, F.Cu at (181.0, 42.1)
- added D11: GREEN, LED_SMD:LED_0805_2012Metric_Pad1.15x1.40mm_HandSolder, F.Cu at (176.2, 45.1)
- added D12: BLUE, LED_SMD:LED_0805_2012Metric_Pad1.15x1.40mm_HandSolder, F.Cu at (172.6, 53.5)
- added D13: PMEG10020ELRX, pandora:D_SOD-123W, F.Cu at (205.2, 67.3)
- added D14: ORANGE, LED_SMD:LED_0805_2012Metric_Pad1.15x1.40mm_HandSolder, F.Cu at (204.1, 71.7)
- added D15: GREEN, LED_SMD:LED_0805_2012Metric_Pad1.15x1.40mm_HandSolder, F.Cu at (210.5, 68.0)
- added D2: 1N4148, Diode_SMD:D_1206_3216Metric_Pad1.42x1.75mm_HandSolder, F.Cu at (102.9, 73.2)
- added D3: 1N4148, Diode_SMD:D_1206_3216Metric_Pad1.42x1.75mm_HandSolder, F.Cu at (92.4, 88.4)
- added D4: 1N4148, Diode_SMD:D_1206_3216Metric_Pad1.42x1.75mm_HandSolder, F.Cu at (102.9, 76.5)
- added D5: 1N4148, Diode_SMD:D_1206_3216Metric_Pad1.42x1.75mm_HandSolder, F.Cu at (102.9, 79.9)
- added D6: RED, LED_SMD:LED_0805_2012Metric_Pad1.15x1.40mm_HandSolder, F.Cu at (167.8, 53.5)
- added D7: GREEN, LED_SMD:LED_0805_2012Metric_Pad1.15x1.40mm_HandSolder, F.Cu at (160.3, 55.5)
- added D8: BLUE, LED_SMD:LED_0805_2012Metric_Pad1.15x1.40mm_HandSolder, F.Cu at (176.2, 42.1)
- added D9: BLUE, LED_SMD:LED_0805_2012Metric_Pad1.15x1.40mm_HandSolder, F.Cu at (165.1, 56.6)
- added F1: 0ZCJ0075FF2E, Fuse:Fuse_1206_3216Metric_Pad1.42x1.75mm_HandSolder, F.Cu at (100.5, 48.5)
- added FB1: 1206_4A, Inductor_SMD:L_1206_3216Metric_Pad1.42x1.75mm_HandSolder, F.Cu at (331.5, -26.7)
- added FB2: 0603_500mA, Inductor_SMD:L_0603_1608Metric_Pad1.05x0.95mm_HandSolder, F.Cu at (189.7, 31.9)
- added FB3: 1206_4A, Inductor_SMD:L_1206_3216Metric_Pad1.42x1.75mm_HandSolder, F.Cu at (206.2, 62.7)
- added H1: M3, MountingHole:MountingHole_3.2mm_M3, F.Cu at (192.9, 52.5)
- added H2: M3, MountingHole:MountingHole_3.2mm_M3, F.Cu at (200.9, 44.5)
- added H3: M3, MountingHole:MountingHole_3.2mm_M3, F.Cu at (192.9, 44.5)
- added H4: M3, MountingHole:MountingHole_3.2mm_M3, F.Cu at (200.9, 52.5)
- added J1: SMA, Connector_Coaxial:SMA_Molex_73251-1153_EdgeMount_Horizontal, F.Cu at (130.7, 79.0)
- added J2: PinHeader_100mil_01x04, Connector_PinHeader_2.54mm:PinHeader_1x04_P2.54mm_Vertical, F.Cu at (163.8, -14.0)
- added J3: JST-SH_2, Connector_JST:JST_SH_SM02B-SRSS-TB_1x02-1MP_P1.00mm_Horizontal, F.Cu at (167.0, 25.7)
- added J4: TX3 / MTA-156-3, pandora:TE_640389-3, F.Cu at (62.4, 55.7)
- added J5: Conn_ARM_JTAG_SWD_10, pandora:PinHeader_2x05_P1.27mm_Vertical_SMD_Long, F.Cu at (11.4, 73.7)
- added J6: USB_B_Mini, pandora:USB_MiniB_KMBSMT5SS30, F.Cu at (79.4, 49.5)
- added JP1: SJ2, Jumper:SolderJumper-2_P1.3mm_Open_Pad1.0x1.5mm, F.Cu at (169.7, 56.8)
- added JP2: SJ2, Jumper:SolderJumper-2_P1.3mm_Open_Pad1.0x1.5mm, F.Cu at (176.0, 48.4)
- added JP3: SJ2, Jumper:SolderJumper-2_P1.3mm_Open_Pad1.0x1.5mm, F.Cu at (180.8, 45.4)
- added JP4: SJ2, Jumper:SolderJumper-2_P1.3mm_Open_Pad1.0x1.5mm, F.Cu at (184.4, 77.9)
- added JP5: SJ2, Jumper:SolderJumper-2_P1.3mm_Open_Pad1.0x1.5mm, F.Cu at (188.8, 77.9)
- added JP6: SJ2_Bridged, Jumper:SolderJumper-2_P1.3mm_Bridged_Pad1.0x1.5mm, F.Cu at (145.9, 15.8)
- added JP7: SJ2, Jumper:SolderJumper-2_P1.3mm_Open_Pad1.0x1.5mm, F.Cu at (104.1, 57.4)
- added JP8: SJ2, Jumper:SolderJumper-2_P1.3mm_Open_Pad1.0x1.5mm, F.Cu at (108.5, 53.0)
- added JP9: SJ2, Jumper:SolderJumper-2_P1.3mm_Open_Pad1.0x1.5mm, F.Cu at (145.9, 19.4)
- added L1: 2.4nH, pandora:0402_HandSoldering, F.Cu at (144.0, 68.8)
- added L2: 2nH, pandora:0402_HandSoldering, F.Cu at (135.5, 77.4)
- added L3: 2nH, pandora:0402_HandSoldering, F.Cu at (147.2, 66.8)
- added L4: 2.4nH, pandora:0402_HandSoldering, F.Cu at (138.6, 75.4)
- added L5: 6.8uH, Inductor_SMD:L_0805_2012Metric_Pad1.15x1.40mm_HandSolder, F.Cu at (182.5, 64.2)
- added L6: 4.7uH, Inductor_SMD:L_Wuerth_MAPI-4020, F.Cu at (252.7, 57.8)
- added NT1: Net-Tie_2, NetTie:NetTie-2_SMD_Pad2.0mm, F.Cu at (195.5, 11.4)
- added NT2: Net-Tie_2, NetTie:NetTie-2_SMD_Pad2.0mm, F.Cu at (191.0, 23.4)
- added NT3: Net-Tie_2, NetTie:NetTie-2_SMD_Pad2.0mm, F.Cu at (182.2, 29.9)
- added NT4: Net-Tie_2, NetTie:NetTie-2_SMD_Pad2.0mm, F.Cu at (195.5, 15.0)
- added NT5: Net-Tie_2, NetTie:NetTie-2_SMD_Pad2.0mm, F.Cu at (183.5, 23.4)
- added Q1: DMP1045U, Package_TO_SOT_SMD:SOT-23_Handsoldering, F.Cu at (199.1, 67.9)
- added R1: 1.2k, Resistor_SMD:R_0603_1608Metric_Pad1.05x0.95mm_HandSolder, F.Cu at (330.2, -47.0)
- added R10: 120k, Resistor_SMD:R_0603_1608Metric_Pad1.05x0.95mm_HandSolder, F.Cu at (283.1, -46.2)
- added R11: 3.3k, Resistor_SMD:R_0603_1608Metric_Pad1.05x0.95mm_HandSolder, F.Cu at (181.4, 50.9)
- added R12: 1.2k, Resistor_SMD:R_0603_1608Metric_Pad1.05x0.95mm_HandSolder, F.Cu at (174.0, 56.3)
- added R13: 330, Resistor_SMD:R_0603_1608Metric_Pad1.05x0.95mm_HandSolder, F.Cu at (178.4, 53.3)
- added R14: 390, Resistor_SMD:R_0603_1608Metric_Pad1.05x0.95mm_HandSolder, F.Cu at (160.1, 58.3)
- added R15: 680, Resistor_SMD:R_0603_1608Metric_Pad1.05x0.95mm_HandSolder, F.Cu at (182.7, 53.4)
- added R16: 560, Resistor_SMD:R_0603_1608Metric_Pad1.05x0.95mm_HandSolder, F.Cu at (177.1, 51.5)
- added R17: 390, Resistor_SMD:R_0603_1608Metric_Pad1.05x0.95mm_HandSolder, F.Cu at (178.4, 56.5)
- added R18: 10, Resistor_SMD:R_1210_3225Metric_Pad1.42x2.65mm_HandSolder, F.Cu at (154.9, 56.1)
- added R19: 10k, Resistor_SMD:R_0603_1608Metric_Pad1.05x0.95mm_HandSolder, F.Cu at (180.1, 69.8)
- added R2: 3.6k, Resistor_SMD:R_0603_1608Metric_Pad1.05x0.95mm_HandSolder, F.Cu at (325.1, -47.0)
- added R20: 100k, Resistor_SMD:R_0603_1608Metric_Pad1.05x0.95mm_HandSolder, F.Cu at (187.0, 63.9)
- added R21: 0, Resistor_SMD:R_0603_1608Metric_Pad1.05x0.95mm_HandSolder, F.Cu at (85.3, 59.5)
- added R22: 0, Resistor_SMD:R_0603_1608Metric_Pad1.05x0.95mm_HandSolder, F.Cu at (80.9, 59.5)
- added R23: 0, Resistor_SMD:R_0603_1608Metric_Pad1.05x0.95mm_HandSolder, F.Cu at (76.6, 59.5)
- added R24: 1k, Resistor_SMD:R_0603_1608Metric_Pad1.05x0.95mm_HandSolder, F.Cu at (213.4, 70.8)
- added R25: 10k, Resistor_SMD:R_0603_1608Metric_Pad1.05x0.95mm_HandSolder, F.Cu at (219.8, 65.3)
- added R26: 10k, Resistor_SMD:R_0603_1608Metric_Pad1.05x0.95mm_HandSolder, F.Cu at (213.4, 73.3)
- added R27: 1k, Resistor_SMD:R_0603_1608Metric_Pad1.05x0.95mm_HandSolder, F.Cu at (217.7, 70.7)
- added R28: 10k, Resistor_SMD:R_0603_1608Metric_Pad1.05x0.95mm_HandSolder, F.Cu at (246.4, 54.0)
- added R3: 10k, Resistor_SMD:R_0603_1608Metric_Pad1.05x0.95mm_HandSolder, F.Cu at (91.6, 91.3)
- added R4: 10k, Resistor_SMD:R_0603_1608Metric_Pad1.05x0.95mm_HandSolder, F.Cu at (108.1, 72.7)
- added R5: 10k, Resistor_SMD:R_0603_1608Metric_Pad1.05x0.95mm_HandSolder, F.Cu at (97.6, 87.9)
- added R6: 10k, Resistor_SMD:R_0603_1608Metric_Pad1.05x0.95mm_HandSolder, F.Cu at (108.1, 75.2)
- added R7: 150k, Resistor_SMD:R_0603_1608Metric_Pad1.05x0.95mm_HandSolder, F.Cu at (293.4, -40.6)
- added R8: 160k, Resistor_SMD:R_0603_1608Metric_Pad1.05x0.95mm_HandSolder, F.Cu at (277.2, -41.6)
- added R9: 150k, Resistor_SMD:R_0603_1608Metric_Pad1.05x0.95mm_HandSolder, F.Cu at (281.6, -41.6)
- added REF**: Li-ion_52x34.5mm_Fancy_Filled, pandora:Bat_52x34.5mm_Zone_Fancy_Filled, B.Cu at (74.9, 130.8)
- added RV1: 10k, Potentiometer_SMD:Potentiometer_Bourns_TC33X_Vertical, F.Cu at (175.7, 86.7)
- added SPK1: DBX-01PN, pandora:DBX-01PN, F.Cu at (158.6, 47.3)
- added SW1: GF-126-0317, pandora:GF-126-0317, F.Cu at (161.7, 16.3)
- added SW10: PTS645-S-H-50-SMTR92-LFS, pandora:SW_Push_PTS645_SMT, F.Cu at (73.7, 67.7)
- added SW11: PTS645-S-H-50-SMTR92-LFS, pandora:SW_Push_PTS645_SMT, F.Cu at (63.2, 82.9)
- added SW12: PTS645-S-H-50-SMTR92-LFS, pandora:SW_Push_PTS645_SMT, F.Cu at (94.7, 82.9)
- added SW13: PTS645-S-M-43-SMTR92-LFS, pandora:SW_Push_PTS645_SMT, F.Cu at (84.2, 67.7)
- added SW14: PTS645-S-K-50-SMTR92-LFS, pandora:SW_Push_PTS645_SMT, F.Cu at (63.2, 90.5)
- added SW15: PTS645-S-K-50-SMTR92-LFS, pandora:SW_Push_PTS645_SMT, F.Cu at (73.7, 82.9)
- added SW16: PTS645-S-K-50-SMTR92-LFS, pandora:SW_Push_PTS645_SMT, F.Cu at (84.2, 75.3)
- added SW17: PTS645-S-K-50-SMTR92-LFS, pandora:SW_Push_PTS645_SMT, F.Cu at (94.7, 67.7)
- added SW18: PTS526-S-K-15-SMTR92-LFS, pandora:SW_Push_PTS526, F.Cu at (164.2, 75.5)
- added SW2: PTS645-S-H-50-SMTR92-LFS, pandora:SW_Push_PTS645_SMT, F.Cu at (84.2, 82.9)
- added SW3: PTS645-S-H-50-SMTR92-LFS, pandora:SW_Push_PTS645_SMT, F.Cu at (94.7, 75.3)
- added SW4: PTS645-S-H-50-SMTR92-LFS, pandora:SW_Push_PTS645_SMT, F.Cu at (105.2, 67.7)
- added SW5: PTS645-S-H-50-SMTR92-LFS, pandora:SW_Push_PTS645_SMT, F.Cu at (84.2, 90.5)
- added SW6: PTS645-S-H-50-SMTR92-LFS, pandora:SW_Push_PTS645_SMT, F.Cu at (63.2, 67.7)
- added SW7: PTS645-S-H-50-SMTR92-LFS, pandora:SW_Push_PTS645_SMT, F.Cu at (73.7, 75.3)
- added SW8: PTS645-S-H-50-SMTR92-LFS, pandora:SW_Push_PTS645_SMT, F.Cu at (73.7, 90.5)
- added SW9: PTS645-S-M-43-SMTR92-LFS, pandora:SW_Push_PTS645_SMT, F.Cu at (63.2, 75.3)
- added TP1: TestPoint, pandora:TestPoint_62-80mil, F.Cu at (104.1, 53.5)
- added TP2: TestPoint, pandora:TestPoint_62-80mil, F.Cu at (110.1, 49.1)
- added TP3: TestPoint, pandora:TestPoint_62-80mil, F.Cu at (141.3, 31.7)
- added TP4: TestPoint, pandora:TestPoint_62-80mil, F.Cu at (99.7, 52.4)
- added TP5: TestPoint, pandora:TestPoint_62-80mil, F.Cu at (105.7, 49.1)
- added TP6: TestPoint, pandora:TestPoint_62-80mil, F.Cu at (94.5, 57.5)
- added TP7: TestPoint, pandora:TestPoint_62-80mil, F.Cu at (146.0, 11.9)
- added TP8: TestPoint, pandora:TestPoint_62-80mil, F.Cu at (99.7, 56.8)
- added TP9: TestPoint, pandora:TestPoint_62-80mil, F.Cu at (90.1, 57.5)
- added U1: LM1086CS-ADJ, Package_TO_SOT_SMD:TO-263-3_TabPin2, F.Cu at (337.8, -41.9)
- added U10: ADM811ZARTZ, Package_TO_SOT_SMD:SOT-143_Handsoldering, F.Cu at (176.1, 65.0)
- added U11: LCD_Adafruit_16x02_Neg_RGB, pandora:LCD_Adafruit_16x02_Neg_RGB, F.Cu at (66.5, 12.3)
- added U12: MCP73831-2-OT, Package_TO_SOT_SMD:SOT-23-5_HandSoldering, F.Cu at (198.8, 72.5)
- added U13: MCP1642D-50, Package_SO:MSOP-8_3x3mm_P0.65mm, F.Cu at (246.4, 57.1)
- added U2: MCP1702T-3302, Package_TO_SOT_SMD:SOT-89-3_Handsoldering, F.Cu at (231.1, -73.0)
- added U3: MCP1702T-3302, Package_TO_SOT_SMD:SOT-89-3_Handsoldering, F.Cu at (231.1, -66.7)
- added U4: MCP6001, Package_TO_SOT_SMD:SOT-23-5_HandSoldering, F.Cu at (293.4, -44.5)
- added U5: MPU-9250, pandora:MPU-9250, F.Cu at (118.5, 92.5)
- added U6: ULN2003D, Package_SO:SOIC-16_3.9x9.9mm_P1.27mm, F.Cu at (237.5, 41.9)
- added U7: 74LCX245, Package_SO:SOIC-20W_7.5x12.8mm_P1.27mm, F.Cu at (76.2, 26.7)
- added U8: CC2652R, pandora:Texas_RGZ0048A, F.Cu at (22.9, 63.5)
- added U9: 74LVC1G08, Package_TO_SOT_SMD:SOT-23-5_HandSoldering, F.Cu at (175.3, 69.2)
- added Y1: NC26_32.768k, pandora:NC26H, F.Cu at (170.5, 69.9)
- added Y2: FA-238_48M, Crystal:Crystal_SMD_SeikoEpson_FA238-4Pin_3.2x2.5mm_HandSoldering, F.Cu at (172.1, 74.8)
Other:
- net class Default: clearance 0.2 -> 0.127; trace_width 0.25 -> 0.254; via_dia 0.8 -> 0.762; via_drill 0.4 -> 0.381
- net class HiPower added: clearance 0.508, trace_width 1.27, via_dia 1.524, via_drill 0.762
- net class Medium added: clearance 0.254, trace_width 0.508, via_dia 0.762, via_drill 0.381
- net class Power added: clearance 0.254, trace_width 0.762, via_dia 1.016, via_drill 0.508
- net class Tight added: clearance 0.127, trace_width 0.2032, via_dia 0.6096, via_drill 0.3048
- rule trace_clearance: 0.2 -> 0.127

Commit message: Begin layout
Parts:
- added H5: M3, MountingHole:MountingHole_3.2mm_M3, F.Cu at (193.0, 61.0)
- added H6: M3, MountingHole:MountingHole_3.2mm_M3, F.Cu at (201.0, 61.0)
- R26, RV1: moved to B.Cu
- moved RV1 124.9 mm to (71.6, 17.8), turned to 90 degrees
- moved D13 43.0 mm to (243.6, 86.6), turned to 90 degrees
- moved Q1 42.7 mm to (236.2, 88.9), turned to 180 degrees
- moved U12 39.3 mm to (236.2, 84.5)
- moved C44 35.3 mm to (240.5, 86.6), turned to 270 degrees
- moved R25 31.5 mm to (236.2, 92.1)
- moved R26 25.7 mm to (236.9, 83.8)
- moved D14 16.1 mm to (208.9, 87.0), turned to 180 degrees
- moved D15 15.9 mm to (208.9, 83.8)
- moved R24 15.6 mm to (213.4, 86.4)
- moved R27 14.4 mm to (213.4, 84.5)
Routing:
- net Net-(R26-Pad2): track 0.00 -> 2.34 mm, vias 0 -> 1
Other:
- net class Default: via_dia 0.762 -> 0.6096; via_drill 0.381 -> 0.3048

Commit message: Continue layout
Parts:
- AE1: footprint pandora:Texas_SWRU120D_InvF_2.4GHz -> pandora:Texas_SWRU120D_InvF_2.4GHz_Left
- C25: footprint pandora:0402_HandSoldering -> pandora:0402_Branch_HandSoldering
- C40, C41: footprint pandora:0402_Branch_HandSoldering -> Capacitor_SMD:C_0603_1608Metric_Pad1.05x0.95mm_HandSolder
- JP7, JP8, JP9: moved to B.Cu
- RV1: moved to F.Cu
- U10: footprint Package_TO_SOT_SMD:SOT-143_Handsoldering -> Package_TO_SOT_SMD:SOT-143
- Y2: footprint Crystal:Crystal_SMD_SeikoEpson_FA238-4Pin_3.2x2.5mm_HandSoldering -> pandora:FA-238
- moved C42 247.9 mm to (-58.7, 82.3)
- moved U10 235.2 mm to (-58.7, 78.2), turned to 180 degrees
- moved SW18 230.3 mm to (-66.0, 79.2), turned to 180 degrees
- moved C41 229.8 mm to (-39.0, 96.1), turned to 270 degrees
- moved C37 229.2 mm to (-42.2, 67.8), turned to 270 degrees
- moved C33 228.3 mm to (-46.2, 77.0)
- moved U9 227.5 mm to (-52.1, 77.2)
- moved C29 225.4 mm to (-38.9, 82.5), turned to 90 degrees
- moved C31 222.5 mm to (-40.4, 67.8), turned to 270 degrees
- moved C34 217.4 mm to (-46.2, 80.0)
- moved C30 215.9 mm to (-35.6, 67.8), turned to 270 degrees
- moved C35 215.1 mm to (-37.3, 82.5), turned to 90 degrees
- moved C36 212.9 mm to (-35.1, 82.5), turned to 90 degrees
- moved Y2 208.9 mm to (-36.3, 88.4), turned to 270 degrees
- moved JP6 199.0 mm to (-46.0, 68.3), turned to 180 degrees
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Connections:
- C1 pad 1: VCC -> VIN
- C1 pad 2: GND -> GNDD
- C10 pad 2: GND -> GNDD
- C11 pad 2: GND -> GNDD
- C12 pad 2: GND -> GNDD
- C13 pad 2: GND -> GNDD
- C14 pad 2: GND -> GNDD
- C2 pad 1: VCC -> VIN
- C2 pad 2: GND -> GNDD
- C21 pad 1: GND -> GNDD
- C28 pad 1: GND -> GNDD
- C29 pad 1: GND -> GNDD
- C29 pad 2: VCC -> VMCU
- C3 pad 1: VCC -> VIN
- C3 pad 2: GND -> GNDD
- C30 pad 1: GND -> GNDD
- C30 pad 2: VCC -> VMCU
- C31 pad 1: GND -> GNDD
- C31 pad 2: VCC -> VMCU
- C32 pad 2: GND -> GNDD
- C33 pad 1: GND -> GNDD
- C33 pad 2: VCC -> VMCU
- C34 pad 1: GND -> GNDD
- C34 pad 2: VCC -> VMCU
- C35 pad 1: GND -> GNDD
- C36 pad 1: GND -> GNDD
- C37 pad 1: GND -> GNDD
- C38 pad 1: GND -> GNDD
- C39 pad 2: GND -> GNDD
- C40 pad 1: GND -> GNDD
- C41 pad 2: GND -> GNDD
- C42 pad 1: VCC -> VMCU
- C42 pad 2: GND -> GNDD
- C43 pad 1: GND -> GNDD
- C43 pad 2: VCC -> VMCU
- C7 pad 1: VCC -> VIN
- C7 pad 2: GND -> GNDD
- C8 pad 2: GND -> GNDD
- C9 pad 2: GND -> GNDD
- D1 pad 2: VCC -> VIN
- D6 pad 2: VCC -> VIN
- FB1 pad 2: VCC -> VIN
- FB2 pad 1: VCC -> VMCU
- J4 pad 1: GND -> GNDD
- J4 pad 2: VCC -> VIN
- J4 pad 3: GND -> GNDD
- J5 pad 3: GND -> GNDD
- J5 pad 5: GND -> GNDD
- JP7 pad 2: GND -> GNDD
- JP8 pad 2: GND -> GNDD
- JP9 pad 2: GND -> GNDD
- NT1 pad 1: GND -> GNDD
- NT1 pad 2: GND -> GNDD
- NT2 pad 1: GND -> GNDD
- NT3 pad 1: GND -> GNDD
- NT4 pad 1: GND -> GNDD
- NT5 pad 1: GND -> GNDD
- R11 pad 2: GND -> GNDD
- R12 pad 2: GND -> GNDD
- R19 pad 1: VCC -> VMCU
- R2 pad 2: GND -> GNDD
- R20 pad 2: GND -> GNDD
- RV1 pad 3: GND -> GNDD
- SW18 pad 1: GND -> GNDD
- TP2 pad 1: VCC -> VIN
- TP7 pad 1: GND -> GNDD
- TP8 pad 1: GND -> GNDD
- U10 pad 1: GND -> GNDD
- U10 pad 4: VCC -> VMCU
- U11 pad 1: GND -> GNDD
- U2 pad 1: GND -> GNDD
- U6 pad 8: GND -> GNDD
- U7 pad 10: GND -> GNDD
- U7 pad 19: GND -> GNDD
- U8 pad 13: VCC -> VMCU
- U8 pad 22: VCC -> VMCU
- U8 pad 34: VCC -> VMCU
- U8 pad 44: VCC -> VMCU
- U8 pad 49: GND -> GNDD
- U9 pad 3: GND -> GNDD
- U9 pad 5: VCC -> VMCU
- Y2 pad 2: GND -> GNDD
- Y2 pad 4: GND -> GNDD

Commit message: Continue layout (CPWG width needs to be defined)
Parts:
- C38, C39, J3: moved to B.Cu
- Y1: footprint pandora:NC26H -> pandora:NC26H_Mirrored
- moved R9 345.2 mm to (-19.8, 119.9)
- moved R7 345.0 mm to (-22.4, 119.9), turned to 270 degrees
- moved R10 344.1 mm to (-17.3, 118.1)
- moved C17 344.0 mm to (-22.4, 111.0), turned to 90 degrees
- moved R8 343.7 mm to (-24.9, 119.9), turned to 270 degrees
- moved U4 343.2 mm to (-21.3, 115.6)
- moved C16 342.8 mm to (-19.8, 111.0), turned to 90 degrees
- moved C43 228.0 mm to (-40.1, 101.6), turned to 90 degrees
- moved C39 213.0 mm to (-40.1, 80.3), turned to 180 degrees
- moved C38 208.6 mm to (-40.1, 77.7)
- moved Y1 208.3 mm to (-37.6, 78.7), turned to 90 degrees
- moved J3 129.2 mm to (61.2, 99.8), turned to 90 degrees
- moved U11 127.3 mm to (-156.0, 40.2)
- moved C28 127.3 mm to (-123.7, 52.1)
- moved JP7 127.3 mm to (-117.9, 45.0)
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Other:
- net class CPWG added: clearance 0.127, trace_width 0.508, via_dia 0.6096, via_drill 0.3048

Commit message: Continue layout
Parts:
- C1, C2, C3, C40, C41, L5: moved to B.Cu
- moved R2 435.8 mm to (-27.5, 209.2), turned to 270 degrees
- moved R1 434.7 mm to (-29.3, 197.5), turned to 270 degrees
- moved U1 430.0 mm to (-21.4, 194.5), turned to 90 degrees
- moved C9 427.6 mm to (-23.2, 209.2)
- moved C8 421.3 mm to (-15.8, 209.2), turned to 270 degrees
- moved FB1 413.3 mm to (-12.8, 202.1), turned to 0 degrees
- moved C11 360.8 mm to (-54.0, 156.0)
- moved C12 360.8 mm to (-42.2, 153.9)
- moved C13 360.8 mm to (-39.4, 153.9)
- moved U2 360.8 mm to (-48.3, 155.3)
- moved H5 336.1 mm to (-130.6, 151.6)
- moved C15 335.6 mm to (-41.4, 118.7), turned to 180 degrees
- moved U3 332.1 mm to (-40.0, 125.1), turned to 90 degrees
- moved C14 329.9 mm to (-39.3, 130.8), turned to 180 degrees
- moved D2 306.6 mm to (-129.3, 104.6), turned to 270 degrees
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Connections:
- C1 pad 2: GNDD -> GNDIN
- C2 pad 2: GNDD -> GNDIN
- C3 pad 2: GNDD -> GNDIN
- C7 pad 2: GNDD -> GNDIN
- J4 pad 1: GNDD -> GNDIN
- J4 pad 3: GNDD -> GNDIN
- NT1 pad 1: GNDD -> GNDIN
- NT2 pad 1: GNDD -> GNDIN
- NT3 pad 1: GNDD -> GNDIN
- NT4 pad 1: GNDD -> GNDIN
- NT5 pad 1: GNDD -> GNDIN
- R11 pad 2: GNDD -> GNDIN
- TP7 pad 1: GNDD -> GNDIN
- U8 pad 10: /keypad/KPD_OUT2 -> /lcd/LCD_DB5
- U8 pad 11: /keypad/KPD_OUT3 -> /lcd/LCD_DB6
- U8 pad 12: /keypad/KPD_OUT4 -> /lcd/LCD_DB7
- U8 pad 14: /lcd/LCD_DB0 -> /keypad/KPD_IN1
- U8 pad 15: /lcd/LCD_DB1 -> /keypad/KPD_IN2
- U8 pad 16: /lcd/LCD_DB2 -> /keypad/KPD_IN3
- U8 pad 17: /lcd/LCD_DB3 -> /keypad/KPD_IN4
- U8 pad 18: /lcd/LCD_DB4 -> /keypad/KPD_OUT1
- U8 pad 19: /lcd/LCD_DB5 -> /keypad/KPD_OUT2
- U8 pad 20: /lcd/LCD_DB6 -> /keypad/KPD_OUT3
- U8 pad 21: /lcd/LCD_DB7 -> /keypad/KPD_OUT4
- U8 pad 38: /imu/IMU_SCK -> /imu/IMU_MISO
- U8 pad 40: /imu/IMU_MISO -> /imu/IMU_SCK
- U8 pad 5: /keypad/KPD_IN1 -> /lcd/LCD_DB0
- U8 pad 6: /keypad/KPD_IN2 -> /lcd/LCD_DB1
- U8 pad 7: /keypad/KPD_IN3 -> /lcd/LCD_DB2
- U8 pad 8: /keypad/KPD_IN4 -> /lcd/LCD_DB3
- U8 pad 9: /keypad/KPD_OUT1 -> /lcd/LCD_DB4
Routing:
- net Net-(D2-Pad2): track 0.00 -> 22.5 mm
- net Net-(C41-Pad1): track 0.00 -> 20.4 mm, vias 0 -> 1
- net /imu/IMU_MISO: track 0.00 -> 19.1 mm, vias 0 -> 2
- net VMCU: track 0.00 -> 18.5 mm
- net Net-(D5-Pad2): track 0.00 -> 17.5 mm
- net /servo/AIN: track 0.00 -> 16.8 mm
- net Net-(R1-Pad2): track 0.00 -> 15.1 mm
- net /imu/IMU_~CS: track 0.00 -> 14.0 mm
- net /imu/IMU_SCK: track 0.00 -> 12.9 mm
- net Net-(C40-Pad2): track 0.00 -> 12.6 mm, vias 0 -> 1
- net /imu/IMU_MOSI: track 0.00 -> 12.3 mm
- net /mcu/VMCUA: track 0.00 -> 11.6 mm
- net Net-(D4-Pad2): track 0.00 -> 6.96 mm
- net Net-(D3-Pad2): track 0.00 -> 6.96 mm
- net /lcd/LCD_DB0: track 0.00 -> 5.27 mm
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- added copper zone on F.Cu, net GNDD
- added copper zone on F.Cu, net Net-(C8-Pad1)
- added copper zone on F.Cu, net Net-(C9-Pad1)
Other:
- net class Default: clearance 0.127 -> 0.2032
- net class Tight: clearance 0.127 -> 0.1524
- rule trace_clearance: 0.127 -> 0.2032
- board text added: "0"
- board text added: "1"
- board text added: "2"
- board text added: "3"
- board text added: "4"
- board text added: "5"
- board text added: "6"
- board text added: "7"
- board text added: "8"
- board text added: "9"
- board text added: "A"
- board text added: "B"
- board text added: "D"
- board text added: "L"
- board text added: "R"
- board text added: "U"

Commit message: Continue layout
Parts:
- R24, R27: moved to B.Cu
- moved D13 316.9 mm to (-67.9, 145.1), turned to 270 degrees
- moved C44 310.7 mm to (-64.6, 145.1), turned to 90 degrees
- moved R26 304.1 mm to (-60.5, 147.9), turned to 180 degrees
- moved U12 302.6 mm to (-59.8, 147.2), turned to 180 degrees
- moved Q1 300.9 mm to (-59.8, 142.6), turned to 0 degrees
- moved R25 299.7 mm to (-59.8, 139.1), turned to 180 degrees
- moved U6 297.9 mm to (-58.0, 79.8), turned to 90 degrees
- moved R24 294.1 mm to (-58.7, 151.0)
- moved D14 293.9 mm to (-63.1, 151.0)
- moved C45 293.2 mm to (-55.2, 145.4), turned to 270 degrees
- moved R27 291.5 mm to (-55.7, 150.0), turned to 90 degrees
- moved C21 289.5 mm to (-50.4, 79.8), turned to 90 degrees
- moved D15 284.0 mm to (-52.1, 151.0), turned to 180 degrees
- moved SW1 250.2 mm to (-61.3, 129.9)
- moved SW14 106.6 mm to (-188.8, 134.0), turned to 45 degrees
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Connections:
- SW1 pad 1: Net-(C9-Pad1) -> VBOOST
- SW1 pad 3: VBOOST -> Net-(C9-Pad1)
- SW1 pad 4: Net-(SW1-Pad4) -> VBAT
- SW1 pad 6: VBAT -> Net-(SW1-Pad6)
Routing:
- net /keypad/KPD_IN4: track 4.93 -> 76.4 mm
- net /keypad/KPD_IN1: track 4.73 -> 72.9 mm
- net Net-(D5-Pad2): track 17.5 -> 73.6 mm
- net /keypad/KPD_IN3: track 4.92 -> 51.7 mm
- net /keypad/KPD_IN2: track 4.66 -> 45.6 mm
- net Net-(C25-Pad3): track 0.00 -> 30.9 mm
- net Net-(D3-Pad2): track 6.96 -> 32.1 mm
- net Net-(D4-Pad2): track 6.96 -> 22.1 mm
- net Net-(R28-Pad1): track 0.00 -> 6.85 mm
- net Net-(C25-Pad1): track 0.00 -> 4.81 mm
- net Net-(C23-Pad2): track 0.00 -> 3.75 mm
- net GNDBAT: track 0.00 -> 3.58 mm
- net Net-(C26-Pad1): track 0.00 -> 3.54 mm
- net Net-(L6-Pad2): track 0.00 -> 3.39 mm
- net Net-(C47-Pad1): track 0.00 -> 1.89 mm
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- added copper zone on F.Cu, net /battery/VLV
- added copper zone on F.Cu, net GNDBAT
- added copper zone on F.Cu, net Net-(C47-Pad1)
- added copper zone on F.Cu, net Net-(L6-Pad2)

Commit message: Continue layout
Parts:
- moved C46 330.6 mm to (-63.8, 141.6)
- moved L6 328.1 mm to (-63.4, 145.7), turned to 90 degrees
- moved R28 319.9 mm to (-58.0, 149.5), turned to 180 degrees
- moved U13 316.2 mm to (-57.0, 146.4), turned to 180 degrees
- moved C47 312.5 mm to (-56.0, 143.2), turned to 180 degrees
- moved C48 311.2 mm to (-55.9, 140.9), turned to 180 degrees
- moved C49 310.0 mm to (-55.9, 138.3), turned to 180 degrees
- moved FB3 304.3 mm to (-52.1, 141.6), turned to 270 degrees
- moved NT1 262.5 mm to (-29.5, 146.7), turned to 270 degrees
- moved FB2 253.3 mm to (-51.6, 108.9), turned to 270 degrees
- moved F1 176.3 mm to (-73.4, 159.8)
- moved J6 176.3 mm to (-73.6, 167.4)
- moved C14 76.5 mm to (-46.4, 118.1), turned to 90 degrees
- moved U3 69.7 mm to (-40.6, 117.5), turned to 0 degrees
- moved C15 67.0 mm to (-41.0, 113.7)
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Connections:
- SW1 pad 1: VBOOST -> Net-(C9-Pad1)
- SW1 pad 3: Net-(C9-Pad1) -> VBOOST
- SW1 pad 4: VBAT -> Net-(SW1-Pad4)
- SW1 pad 6: Net-(SW1-Pad6) -> VBAT
Routing:
- net /connectors/JTAG_TDI: track 0.00 -> 11.1 mm
- net VBOOST: track 0.00 -> 9.57 mm
- net Net-(C9-Pad1): track 0.00 -> 5.16 mm
- net Net-(R1-Pad2): track 15.1 -> 18.0 mm
- net Net-(L6-Pad2): track 3.39 -> 4.59 mm
- added copper zone on F.Cu, net +3.3VA
- added copper zone on F.Cu, net +3V3
- added copper zone on F.Cu, net +5V
- added copper zone on F.Cu, net GNDA
- removed copper zone on F.Cu, net Net-(L6-Pad2)
Other:
- board text added: "JLCJLCJLCJLC"

Commit message: Continue layout
Parts:
- C16, C17, C4, C42, C43, C44, C45, C5, C6, R11, R12, R25: moved to B.Cu
- Q1: footprint Package_TO_SOT_SMD:SOT-23_Handsoldering -> Package_TO_SOT_SMD:SOT-23
- U12, U4, U9: footprint Package_TO_SOT_SMD:SOT-23-5_HandSoldering -> Package_TO_SOT_SMD:SOT-23-5
- U2, U3: footprint Package_TO_SOT_SMD:SOT-89-3_Handsoldering -> Package_TO_SOT_SMD:SOT-89-3
- moved R11 223.4 mm to (-26.3, 133.1), turned to 270 degrees
- moved R12 218.3 mm to (-30.3, 133.1), turned to 90 degrees
- moved D6 209.7 mm to (-26.3, 133.1), turned to 270 degrees
- moved D7 205.9 mm to (-30.3, 133.1), turned to 90 degrees
- moved TP2 166.3 mm to (-29.0, 140.2)
- moved TP7 165.8 mm to (-29.0, 144.5)
- moved J3 132.9 mm to (-68.4, 129.1), turned to 0 degrees
- moved REF** 62.7 mm to (33.8, 178.1)
- moved C12 59.6 mm to (-53.0, 112.3)
- moved C13 59.6 mm to (-53.0, 109.7)
- moved U2 59.6 mm to (-52.7, 116.1)
- moved C11 59.6 mm to (-56.9, 115.3)
- moved D13 52.6 mm to (-69.7, 123.5), turned to 180 degrees
- moved C45 48.3 mm to (-60.3, 126.8), turned to 90 degrees
- moved JP6 48.2 mm to (-65.6, 88.8)
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Connections:
- C18 pad 2: GND -> GNDD
- C19 pad 1: GND -> GNDD
- C20 pad 1: GND -> GNDD
- U5 pad 11: GND -> GNDD
- U5 pad 18: GND -> GNDD
- U5 pad 20: GND -> GNDD
Routing:
- net VCHG: track 0.00 -> 27.1 mm, vias 0 -> 2
- net /battery/VLV: track 1.89 -> 20.9 mm, vias 0 -> 2
- net GNDBAT: track 3.58 -> 20.2 mm, vias 0 -> 3
- net Net-(R24-Pad2): track 0.00 -> 11.7 mm, vias 0 -> 1
- net Net-(C45-Pad1): track 0.00 -> 11.1 mm
- net GNDD: track 0.00 -> 10.4 mm, vias 0 -> 7
- net /servo/AIN: track 16.8 -> 26.2 mm
- net VMCU: track 18.5 -> 24.9 mm, vias 0 -> 1
- net Net-(F1-Pad1): track 0.00 -> 6.16 mm
- net +3.3VA: track 0.00 -> 5.49 mm, vias 0 -> 1
- net VBAT: track 0.00 -> 4.72 mm
- net Net-(D15-Pad2): track 0.00 -> 3.44 mm, vias 0 -> 1
- net Net-(D14-Pad1): track 0.00 -> 2.90 mm, vias 0 -> 1
- net Net-(R10-Pad2): track 0.00 -> 2.85 mm
- net /imu/IMU_MISO: track 19.1 -> 16.3 mm
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Other:
- net class CPWG: trace_width 0.508 -> 0.6096; via_dia 0.6096 -> 0.762; via_drill 0.3048 -> 0.381
- net class Default: via_dia 0.6096 -> 0.762; via_drill 0.3048 -> 0.381
- net class Tight: via_dia 0.6096 -> 0.762; via_drill 0.3048 -> 0.381
- rule trace_min: 0.2 -> 0.1524
- rule via_min_drill: 0.3 -> 0.3048
- rule via_min_size: 0.4 -> 0.6096
- board text added: "5V"
- board text added: "BATT"
- board text added: "CHG"
- board text added: "DONE"
- board text added: "EXT"
- board text added: "FDBK"
- board text added: "GND"
- board text added: "PWM"
- board text added: "V+"
- board text added: "VIN"
